File: VCO/VCO.kicad_pcb (KiCad board)
At the start: 2 copper layers, 39 x 110 mm, 59 parts, among them J1 PWM, J2 1V_A, J3 FM, J4 SYNC, J5 POWER, J6 TRI, J7 SQR, J8 Bus_i, J9 Bus_o, Q1 BC847BPN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

Commit message: rev1 updates
Parts:
- removed REF**: OSHW-Logo2_14.6x12mm_SilkScreen, Symbol:OSHW-Logo2_14.6x12mm_SilkScreen
- C10, C3, C4, C5, C6, C8, C9: footprint Capacitor_SMD:C_0805_2012Metric -> Capacitor_SMD:C_0402_1005Metric
- moved R6 7.22 mm to (-24.0, -58.5), turned to 270 degrees
- moved C10 3.75 mm to (-12.5, -60.5)
- moved Q2 2.76 mm to (-27.5, -54.2), turned to 90 degrees
- moved R10 2.63 mm to (-24.7, -46.2)
- moved C8 1.27 mm to (-14.8, -39.2), turned to 90 degrees
- moved C6 0.92 mm to (-23.5, -48.5)
- moved C9 0.72 mm to (-23.8, -39.2)
- moved C4 0.72 mm to (-23.5, -66.5)
- moved C5 0.69 mm to (-14.5, -48.8)
- moved C3 0.57 mm to (-14.5, -70.3)
Connections:
- U2 pad 10: Net-(U2-Pad10) -> GND
- U3 pad 10: Net-(U3-Pad10) -> GND
- U3 pad 8: Net-(U3-Pad10) -> Net-(U3-Pad8)
- U3 pad 9: GND -> Net-(U3-Pad8)
Routing:
- net /PWM_norm: track 130.4 -> 89.4 mm, vias 2 -> 3
- net -12V: track 146.4 -> 121.9 mm, vias 6 -> 0
- net +12V: track 229.9 -> 245.1 mm, vias 7 -> 1
- net /tri2sqr: track 27.4 -> 14.3 mm, vias 0 -> 2
- net /PWM: track 13.3 -> 21.1 mm, vias 0 -> 2
- net Net-(U3-Pad10): track 5.39 -> 0.00 mm
- net GND: track 27.2 -> 22.3 mm, vias 16 -> 18
- net /SQR: track 41.2 -> 45.8 mm, vias 0 -> 2
- net /FM_lin: track 57.8 -> 61.2 mm, vias 1 -> 2
- net Net-(C7-Pad1): track 8.26 -> 5.41 mm
- net Net-(D2-Pad1): track 22.2 -> 24.0 mm
- net /1V_norm: track 41.1 -> 42.7 mm
- net Net-(R1-Pad2): track 65.7 -> 67.2 mm
- net Net-(C10-Pad1): track 3.02 -> 1.61 mm
- net Net-(U3-Pad8): track 0.00 -> 1.27 mm
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Other:
- net class Default: via_dia 0.8 -> 0.6; via_drill 0.4 -> 0.35
- net class Power: trace_width 0.9 -> 0.6
- board text added: "REV1"

Commit message: rev 2 changes, see revision_log
Parts:
- removed J8: Bus_i, Connector_PinHeader_2.54mm:PinHeader_1x04_P2.54mm_Vertical
- removed J9: Bus_o, Connector_PinHeader_2.54mm:PinHeader_1x04_P2.54mm_Vertical
- added G***: LOGO, user-artwork:smiley, F.Cu at (-7.24, -100.5)
- C10, C3, C4, C5, C6, C8, C9: footprint Capacitor_SMD:C_0402_1005Metric -> Capacitor_SMD:C_0603_1608Metric
- Q2: value J112 -> MMBFJ112; footprint user-footprints:TO-92_J112 -> Package_TO_SOT_SMD:SOT-23
- moved Q2 2.76 mm to (-24.8, -54.0)
- moved R10 0.90 mm to (-24.7, -45.4)
- moved C6 0.58 mm to (-23.8, -48.0)
- moved C10 0.56 mm to (-11.9, -60.5)
- moved C9 0.42 mm to (-24.1, -39.5)
- moved C5 0.36 mm to (-14.2, -48.6)
- moved C4 0.36 mm to (-23.8, -66.3)
- moved C3 0.33 mm to (-14.2, -70.1)
- moved C8 0.33 mm to (-14.4, -39.4)
Connections:
- J1 pad TN: /PWM_norm -> GND
- J2 pad TN: /1V_norm -> GND
- J3 pad TN: /FM_norm -> GND
- R6 pad 2: Net-(Q2-PadG) -> Net-(Q2-Pad3)
- RV4 pad 3: Net-(Q2-PadG) -> Net-(Q2-Pad3)
Routing:
- net /PWM_norm: track 89.4 -> 0.00 mm, vias 3 -> 0
- net Net-(Q2-Pad3): track 0.00 -> 68.2 mm, vias 0 -> 2
- net /TRI_norm: track 67.7 -> 0.00 mm, vias 1 -> 0
- net /FM_norm: track 60.2 -> 0.00 mm, vias 1 -> 0
- net /SQR_norm: track 58.9 -> 0.00 mm, vias 1 -> 0
- net Net-(Q2-PadG): track 53.8 -> 0.00 mm, vias 2 -> 0
- net /1V_norm: track 42.7 -> 0.00 mm
- net Net-(J8-Pad2): track 36.0 -> 0.00 mm, vias 2 -> 0
- net -12V: track 121.9 -> 155.1 mm
- net /SQR: track 45.8 -> 68.4 mm
- net GND: track 22.3 -> 28.0 mm, vias 18 -> 16
- net /TRI: track 54.1 -> 59.6 mm
- net /PWM: track 21.1 -> 16.1 mm, vias 2 -> 0
- net /FM_lin: track 61.2 -> 63.6 mm
- net Net-(R1-Pad2): track 67.2 -> 68.8 mm
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Other:
- board text added: "REV2"
- board text removed: "1V"
- board text removed: "FM"
- board text removed: "IN"
- board text removed: "OUT"
- board text removed: "PWM"
- board text removed: "REV1"
- board text removed: "SQR"
- board text removed: "TRI"
- board text removed: "thru"

Commit message: rev 3, see revision log
Parts:
- added C11: 330pF, Capacitor_SMD:C_0805_2012Metric, F.Cu at (-19.2, -73.8)
- added C12: 330pF, Capacitor_SMD:C_0805_2012Metric, F.Cu at (-12.0, -42.8)
- added C13: 4.7pF, Capacitor_SMD:C_0805_2012Metric, F.Cu at (-12.0, -36.0)
- J2: value 1V_A -> 1V
- R1: value 56K -> 91K
- RV5: value 100KT* -> 20KT
- moved R22 2.37 mm to (-9.00, -43.8)
- moved R14 2.30 mm to (-9.00, -41.5)
- moved R18 2.25 mm to (-9.00, -36.8)
- moved R23 2.25 mm to (-9.00, -34.5)
- moved R24 2.25 mm to (-6.00, -36.8)
Connections:
- net /1V_A renamed /1V
- net /FM_lin renamed /FM
- net /Iabc renamed /Iexp
- net /V_expo renamed /Vlin
Routing:
- net /tri2sqr: track 14.3 -> 17.8 mm
- net /TRI: track 59.6 -> 56.7 mm
- net Net-(C11-Pad1): track 9.82 -> 12.5 mm
- net Net-(C13-Pad2): track 5.08 -> 7.43 mm
- net Net-(C12-Pad2): track 4.99 -> 7.28 mm
- net Net-(C11-Pad2): track 9.87 -> 12.1 mm
- net /SQR: track 68.4 -> 66.1 mm
- net Net-(C13-Pad1): track 4.97 -> 7.17 mm
Other:
- board text added: "REV3"
- board text removed: "REV2"
