File: VCO/VCO.kicad_pcb (KiCad board)
At the start: 2 copper layers, 39 x 110 mm, 57 parts, among them J1 PWM, J2 1V_A, J3 FM, J4 SYNC, J5 POWER, J6 TRI, J7 SQR, Q1 BC847BPN, Q2 MMBFJ112, U1 TL072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

Commit message: rev 3 updates, see revision log
Parts:
- removed G***: LOGO, user-artwork:smiley
- D3: footprint user-footprints:LED_3mm -> LED_THT:LED_D3.0mm
- J1, J2, J3, J4, J6, J7: footprint user-footprints:AudioJack_QuPing_Pushfit -> user-main:AudioJack_QingPu_WQP-PJ301BM_Vertical
- R1: value 56K -> 91K; footprint Resistor_SMD:R_0805_2012Metric -> Resistor_SMD:R_0603_1608Metric
- RV4: moved to F.Cu
- RV5: value 100KT* -> 20KT*; moved to F.Cu
- moved RV5 6.99 mm to (-9.54, -32.6)
- moved RV4 6.49 mm to (-21.7, -32.6)
- moved C8 1.52 mm to (-14.4, -40.9)
- moved C9 1.52 mm to (-24.1, -41.0)
- moved R14 1.52 mm to (-11.2, -43.5)
- moved R15 1.52 mm to (-31.0, -38.5)
- moved R16 1.52 mm to (-27.2, -36.3)
- moved R17 1.52 mm to (-27.2, -38.5)
- moved R18 1.52 mm to (-11.2, -38.3)
- moved R19 1.52 mm to (-14.2, -44.3)
- moved R20 1.52 mm to (-14.2, -37.5)
- moved R21 1.52 mm to (-24.2, -37.0)
- moved R22 1.52 mm to (-11.2, -46.0)
- moved R23 1.52 mm to (-11.2, -36.0)
- moved R24 1.52 mm to (-8.25, -38.3)
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Connections:
- J4 pad TN: Net-(J4-PadTN) -> unconnected-(J4-PadTN)
- J6 pad TN: /TRI_norm -> unconnected-(J6-PadTN)
- J7 pad TN: /SQR_norm -> unconnected-(J7-PadTN)
- RV4 pad 1: Net-(RV4-Pad1) -> unconnected-(RV4-Pad1)
- RV5 pad 1: Net-(R1-Pad2) -> unconnected-(RV5-Pad1)
- RV5 pad 3: Net-(RV5-Pad3) -> Net-(R1-Pad2)
- U2 pad 15: Net-(U2-Pad15) -> unconnected-(U2-Pad15)
- U2 pad 2: Net-(U2-Pad2) -> unconnected-(U2-Pad2)
- U2 pad 9: Net-(U2-Pad9) -> unconnected-(U2-Pad9)
Routing:
- net /PWM: track 16.1 -> 23.2 mm, vias 0 -> 2
- net GND: track 28.0 -> 33.6 mm
- net /SYNC: track 33.5 -> 28.9 mm, vias 0 -> 1
- net /SQR: track 68.4 -> 71.7 mm
- net /TRI: track 59.6 -> 62.3 mm
- net Net-(Q2-Pad3): track 68.2 -> 70.5 mm
- net +12V: track 244.4 -> 242.8 mm
- net /PW: track 11.9 -> 10.4 mm
- net /LED: track 12.6 -> 14.1 mm
- net /TRI_raw: track 20.6 -> 19.7 mm
Other:
- net class Default removed
- net class Power removed
- board text added: "100K"
- board text added: "20K"
- board text added: "VCO V1.3 12/30/2021"
- board text removed: "REV2"
