File: Wavefolder/Wavefolder.kicad_pcb (KiCad board)
At the start: 2 copper layers, 28 x 110 mm, 85 parts, among them J1 CV_in, J2 input, J5 fold, J6 pulse, J7 POWER, Q1 MMBT3904, Q2 MMBT3904, U1 TL074, U2 TL074, U3 TL072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

Commit message: rev 3, see revision log
Parts:
- added C15: 220pF, Capacitor_SMD:C_0805_2012Metric, F.Cu at (-6.75, -87.8)
- added C16: 22pF, Capacitor_SMD:C_0805_2012Metric, F.Cu at (-7.00, -28.5)
- U3, U4: value TL072 -> LM358
- moved R9 2.50 mm to (-4.75, -28.5)
- moved R3 1.95 mm to (-4.50, -85.8), turned to 90 degrees
Routing:
- net postfold: track 26.5 -> 24.0 mm
- net Net-(C15-Pad2): track 13.2 -> 15.7 mm
- net Net-(C16-Pad2): track 4.48 -> 6.92 mm
- net Net-(C16-Pad1): track 11.3 -> 13.5 mm
