File: VCO/Panel/vco_panel.kicad_pcb (KiCad board)
At the start: 2 copper layers, 40.3 x 128.5 mm, 14 parts

Commit message: rev 3 updates, see revision log
Parts:
- removed the screwhole* at (2.54, -32.6)
- removed the screwhole* at (15.3, -32.6)
- screwhole* (x2): footprint user-panel:Screw_3M_Slot -> user-panel:Screw_3M_Hole
Other:
- net class Default removed
