File: Wavefolder/Panel/wavefolder_panel.kicad_pcb (KiCad board)
At the start: 2 copper layers, 30 x 128.5 mm, 9 parts

Commit message: rev 3 updates, see revision log
Parts:
- screwhole* (x2): footprint user-panel:Screw_3M_Slot -> user-panel:Screw_3M_Hole
Other:
- net class Default removed
